Commit message: add inertia, mesh

File: ouster_description/urdf/OS1-64.urdf.xacro (robot description, xacro)
@@ -48,5 +48,5 @@
         <sensor type="gpu_ray" name="${name}-OS1-64">
           <pose>0 0 0 0 0 0</pose>
-          <visualize>false</visualize>
+          <visualize>true</visualize>
           <update_rate>${hz}</update_rate>
           <ray>

File: ouster_description/urdf/OSDome-64.urdf.xacro (robot description, xacro)
@@ -2,5 +2,5 @@
 <robot xmlns:xacro="http://www.ros.org/wiki/xacro" name="OSDome-64">
   <xacro:property name="M_PI" value="3.1415926535897931" />
-  <xacro:macro name="OSDome-64" params="*origin parent:=base_link name:=osdome_sensor topic_points:=/osdome_cloud_node/points topic_imu:=/osdome_cloud_node/imu hz:=10 lasers:=64 samples:=512 min_range:=0.5 max_range:=40.0 noise:=0.008 min_angle:=-${M_PI} max_angle:=${M_PI} lidar_link:=osdome_lidar imu_link:=osdome_imu vfov_min:=-1.4835 vfov_max:=0.0 gpu:=false">
+  <xacro:macro name="OSDome-64" params="*origin parent:=base_link name:=osdome_sensor topic_points:=/osdome_cloud_node/points topic_imu:=/osdome_cloud_node/imu hz:=10 lasers:=64 samples:=1024 min_range:=0.5 max_range:=40.0 noise:=0.008 min_angle:=-${M_PI} max_angle:=${M_PI} lidar_link:=osdome_lidar imu_link:=osdome_imu vfov_min:=0.0 vfov_max:=1.4835 gpu:=false">
     <joint name="${name}_mount_joint" type="fixed">
       <xacro:insert_block name="origin" />
@@ -10,19 +10,19 @@
     <link name="${name}">
       <inertial>
-         <mass value="0.33"/>
-         <origin xyz="0 0 0.0365" rpy="0 0 0" />
-         <inertia ixx="0.000241148" ixy="0" ixz="0"
-          iyy="0.000241148" iyz="0" izz="0.000264"/>
+         <mass value="0.47"/>
+         <origin xyz="0 0 0.04" rpy="0 0 0" />
+         <inertia ixx="0.00030456" ixy="0" ixz="0"
+          iyy="0.00030456" iyz="0" izz="0.000437"/>
       </inertial>
       <collision name="base_collision">
-         <origin xyz="0 0 0.0365" rpy="0 0 0" />
+         <origin xyz="0 0 0.042635" rpy="0 0 0" />
          <geometry>
- 	        <cylinder radius="0.04" length="0.073"/>
+ 	        <cylinder radius="0.036" length="0.08527"/>
          </geometry>
       </collision>
       <visual name="base_visual">
-         <origin xyz="0 0 0.0" rpy="0 0 1.5707" />
+         <origin xyz="0 0 0" rpy="0 0 0" />
          <geometry>
-	         <mesh filename="package://ouster_description/meshes/os1_64.dae" />
+	         <mesh filename="package://ouster_description/meshes/osdome_64.dae" />
            <!-- <cylinder length="0.073" radius="0.04" /> -->
          </geometry>
@@ -41,9 +41,8 @@
       <parent link="${name}" />
       <child link="${lidar_link}" />
-      <!--<origin xyz="0.0 0.0 0.03618" rpy="3.14159 0 0" />-->
-      <origin xyz="0.0 0.0 0.03618" rpy="0 0 0" />
+      <origin xyz="0.0 0.0 0.047824" rpy="0 0 0" />
     </joint>
     <!-- Gazebo requires the ouster_gazebo_plugins package -->
-    <gazebo reference="${name}">
+    <gazebo reference="${lidar_link}">
       <xacro:if value="${gpu}">
         <sensor type="gpu_ray" name="${name}-OSDome-64">
@@ -69,5 +68,5 @@
               <min>${min_range}</min>
               <max>${max_range}</max>
-              <resolution>0.03</resolution>
+              <resolution>0.01</resolution>
             </range>
           </ray>
@@ -104,5 +103,5 @@
               <min>${min_range}</min>
               <max>${max_range}</max>
-              <resolution>0.03</resolution>
+              <resolution>0.01</resolution>
             </range>
           </ray>

File: ouster_description/urdf/example_osdome-64.urdf.xacro (robot description, xacro)
@@ -31,6 +31,6 @@
   </link>
   <xacro:include filename="$(find ouster_description)/urdf/OSDome-64.urdf.xacro"/>
-  <OSDome-64 parent="base_link" name="osdome_sensor" hz="10" samples="220" gpu="${gpu}">
-    <origin xyz="0 0 3.0" rpy="0 0 0" />
+  <OSDome-64 parent="base_link" name="osdome_sensor" hz="10" samples="512" gpu="${gpu}">
+    <origin xyz="0 0 2.0" rpy="3.1415926 0 0" />
   </OSDome-64>
 </robot>
