Commit message: add gpu_ray, time field and OSDome

File: ouster_description/urdf/OSDome-64.urdf.xacro (robot description, xacro)
@@ -1,6 +1,6 @@
 <?xml version="1.0"?>
-<robot xmlns:xacro="http://www.ros.org/wiki/xacro" name="OS1-64">
+<robot xmlns:xacro="http://www.ros.org/wiki/xacro" name="OSDome-64">
   <xacro:property name="M_PI" value="3.1415926535897931" />
-  <xacro:macro name="OS1-64" params="*origin parent:=base_link name:=os1_sensor topic_points:=/os1_cloud_node/points topic_imu:=/os1_cloud_node/imu hz:=10 lasers:=64 samples:=512 min_range:=0.9 max_range:=75.0 noise:=0.008 min_angle:=-${M_PI} max_angle:=${M_PI} lidar_link:=os1_lidar imu_link:=os1_imu vfov_min:=-.26 vfov_max:=.26 gpu:=false">
+  <xacro:macro name="OSDome-64" params="*origin parent:=base_link name:=osdome_sensor topic_points:=/osdome_cloud_node/points topic_imu:=/osdome_cloud_node/imu hz:=10 lasers:=64 samples:=512 min_range:=0.5 max_range:=40.0 noise:=0.008 min_angle:=-${M_PI} max_angle:=${M_PI} lidar_link:=osdome_lidar imu_link:=osdome_imu vfov_min:=-1.4835 vfov_max:=0.0 gpu:=false">
     <joint name="${name}_mount_joint" type="fixed">
       <xacro:insert_block name="origin" />
@@ -41,4 +41,5 @@
       <parent link="${name}" />
       <child link="${lidar_link}" />
+      <!--<origin xyz="0.0 0.0 0.03618" rpy="3.14159 0 0" />-->
       <origin xyz="0.0 0.0 0.03618" rpy="0 0 0" />
     </joint>
@@ -46,5 +47,5 @@
     <gazebo reference="${name}">
       <xacro:if value="${gpu}">
-        <sensor type="gpu_ray" name="${name}-OS1-64">
+        <sensor type="gpu_ray" name="${name}-OSDome-64">
           <pose>0 0 0 0 0 0</pose>
           <visualize>false</visualize>
@@ -81,5 +82,5 @@
       </xacro:if>
       <xacro:unless value="${gpu}">
-        <sensor type="ray" name="${name}-OS1-64">
+        <sensor type="ray" name="${name}-OSDome-64">
           <pose>0 0 0 0 0 0</pose>
           <visualize>false</visualize>

File: ouster_description/urdf/example_osdome-64.urdf.xacro (robot description, xacro)
@@ -1,4 +1,6 @@
 <?xml version="1.0"?>
-<robot xmlns:xacro="http://www.ros.org/wiki/xacro" name="os1_example">
+<robot xmlns:xacro="http://www.ros.org/wiki/xacro" name="osdome_example">
+  <xacro:arg name="gpu" default="false"/>
+  <xacro:property name="gpu" value="$(arg gpu)" />
   <!-- Base Footprint -->
   <link name="base_footprint" />
@@ -28,7 +30,7 @@
     </inertial>
   </link>
-  <xacro:include filename="$(find ouster_description)/urdf/OS1-64.urdf.xacro"/>
-  <OS1-64 parent="base_link" name="os1_sensor" hz="10" samples="220">
-    <origin xyz="0 0 1.2" rpy="0 0 0" />
-  </OS1-64>
+  <xacro:include filename="$(find ouster_description)/urdf/OSDome-64.urdf.xacro"/>
+  <OSDome-64 parent="base_link" name="osdome_sensor" hz="10" samples="220" gpu="${gpu}">
+    <origin xyz="0 0 3.0" rpy="0 0 0" />
+  </OSDome-64>
 </robot>

Commit message: modify min_range

File: ouster_description/urdf/OSDome-64.urdf.xacro (robot description, xacro)
@@ -2,5 +2,5 @@
 <robot xmlns:xacro="http://www.ros.org/wiki/xacro" name="OSDome-64">
   <xacro:property name="M_PI" value="3.1415926535897931" />
-  <xacro:macro name="OSDome-64" params="*origin parent:=base_link name:=osdome_sensor topic_points:=/osdome_cloud_node/points topic_imu:=/osdome_cloud_node/imu hz:=10 lasers:=64 samples:=1024 min_range:=0.5 max_range:=40.0 noise:=0.008 min_angle:=-${M_PI} max_angle:=${M_PI} lidar_link:=osdome_lidar imu_link:=osdome_imu vfov_min:=0.0 vfov_max:=1.4835 gpu:=false">
+  <xacro:macro name="OSDome-64" params="*origin parent:=base_link name:=osdome_sensor topic_points:=/osdome_cloud_node/points topic_imu:=/osdome_cloud_node/imu hz:=10 lasers:=64 samples:=1024 min_range:=0.04 max_range:=40.0 noise:=0.008 min_angle:=-${M_PI} max_angle:=${M_PI} lidar_link:=osdome_lidar imu_link:=osdome_imu vfov_min:=0.0 vfov_max:=1.4835 gpu:=false">
     <joint name="${name}_mount_joint" type="fixed">
       <xacro:insert_block name="origin" />

File: ouster_description/urdf/example_osdome-64.urdf.xacro (robot description, xacro)
@@ -32,5 +32,6 @@
   <xacro:include filename="$(find ouster_description)/urdf/OSDome-64.urdf.xacro"/>
   <OSDome-64 parent="base_link" name="osdome_sensor" hz="10" samples="512" gpu="${gpu}">
-    <origin xyz="0 0 2.0" rpy="3.1415926 0 0" />
+    <origin xyz="0 0 2.0" rpy="0 3.1415926 0" />
+    <!--<origin xyz="0 0 2.0" rpy="1.570796 0 0" />-->
   </OSDome-64>
 </robot>

Commit message: modified beam origin and min_range

File: ouster_description/urdf/OSDome-64.urdf.xacro (robot description, xacro)
@@ -2,5 +2,5 @@
 <robot xmlns:xacro="http://www.ros.org/wiki/xacro" name="OSDome-64">
   <xacro:property name="M_PI" value="3.1415926535897931" />
-  <xacro:macro name="OSDome-64" params="*origin parent:=base_link name:=osdome_sensor topic_points:=/osdome_cloud_node/points topic_imu:=/osdome_cloud_node/imu hz:=10 lasers:=64 samples:=1024 min_range:=0.04 max_range:=40.0 noise:=0.008 min_angle:=-${M_PI} max_angle:=${M_PI} lidar_link:=osdome_lidar imu_link:=osdome_imu vfov_min:=0.0 vfov_max:=1.4835 gpu:=false">
+  <xacro:macro name="OSDome-64" params="*origin parent:=base_link name:=osdome_sensor topic_points:=/osdome_cloud_node/points topic_imu:=/osdome_cloud_node/imu hz:=10 lasers:=64 samples:=1024 min_range:=0.001 max_range:=40.0 noise:=0.008 min_angle:=-${M_PI} max_angle:=${M_PI} lidar_link:=osdome_lidar imu_link:=osdome_imu vfov_min:=0 vfov_max:=1.4835 gpu:=false">
     <joint name="${name}_mount_joint" type="fixed">
       <xacro:insert_block name="origin" />
@@ -41,5 +41,6 @@
       <parent link="${name}" />
       <child link="${lidar_link}" />
-      <origin xyz="0.0 0.0 0.047824" rpy="0 0 0" />
+      <!--<origin xyz="0.0 0.0 0.047824" rpy="0 0 0" />-->
+      <origin xyz="0.0 0.0 0.08527" rpy="0 0 0" />
     </joint>
     <!-- Gazebo requires the ouster_gazebo_plugins package -->
